File: hardware/stm32-nema17-servo.kicad_pcb (KiCad board)
At the start: 2 copper layers, 48 x 43.9 mm, 97 parts, among them J1 Conn_01x05, J2 C31-S-RA-CS1A-BK-SS, J3 TC-2050, J4 Screw_Terminal_01x02, J5 Screw_Terminal_01x02, J7 Conn_01x03, J8 Conn_01x03, J9 Conn_01x02, M1 Stepper_Motor_bipolar, Q1 NVTFS5C658NL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

Commit message: hardware v0.3 as ordered
Parts:
- removed U2: 74LVC2G32, Package_SON:X2SON-8_1.4x1mm_P0.35mm
- added R33: 1K, Resistor_SMD:R_0402_1005Metric, F.Cu at (162.1, 115.0)
- added R34: 1K, Resistor_SMD:R_0402_1005Metric, F.Cu at (163.1, 115.0)
- moved R27 0.28 mm to (157.9, 103.1)
- moved R32 0.10 mm to (141.6, 113.0)
Connections:
- U4 pad 1: A_NSS -> ASEL
- U6 pad 32: DRV_NSS -> DRVSEL
Routing:
- net A_NSS: track 37.3 -> 0.00 mm, vias 4 -> 0
- net ASEL: track 4.55 -> 36.1 mm, vias 0 -> 2
- net DRVSEL: track 7.30 -> 36.2 mm, vias 2 -> 4
- net DRV_NSS: track 28.0 -> 0.00 mm, vias 2 -> 0
- net VBUSDIV: track 48.6 -> 28.3 mm, vias 6 -> 4
- net VDD: track 95.3 -> 106.7 mm
- net SPI_NSS: track 6.87 -> 4.62 mm, vias 2 -> 0
- net +3V3: track 60.5 -> 58.7 mm
- net SWDIO: track 8.97 -> 7.90 mm
- net SLCK: track 38.3 -> 37.8 mm
- net GND: track 105.6 -> 105.2 mm, vias 58 -> 57
Other:
- board text added: "SW1"
- board text removed: "RST"
