File: hardware/stm32-nema17-servo.sch (KiCad schematic (older format))
At the start: 98 parts, among them J1 Conn_01x05, J2 C31-S-RA-CS1A-BK-SS, J3 TC-2050, J4 Screw_Terminal_01x02, J5 Screw_Terminal_01x02, J7 Conn_01x03, J8 Conn_01x03, J9 Conn_01x02, M1 Stepper_Motor_bipolar, Q1 NVTFS5C658NL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

Commit message: cosmetic updates to schematic and board
Parts:
- Q10, Q8, Q9: MPN (none) -> SSM3K35CTC
- R33, R34: MPN RC0402JR-07680RL -> RC0402FR-071KL
- U1: MPN (none) -> STM32G431CBU
- U3: MPN (none) -> UCC27516
- U4: MPN (none) -> AS5047D
- U5: MPN (none) -> TPS62172DSG
- U6: MPN (none) -> DRV8323RS
Changed lines of the file:
@@
 F 2 "stm32-nema17:TSSOP-14_4.4x5mm_P0.65mm-inlaid" H 5000 1200 50  0001 C CNN
 F 3 "https://ams.com/documents/20143/36005/AS5047D_DS000394_2-00.pdf/c7225c06-112f-82c5-4471-17a2711a7f0e" H 3850 1700 50  0001 C CNN
+F 4 "AS5047D" H 4100 1750 50  0001 C CNN "MPN"
 	1    4100 1750
 	1    0    0    -1
@@
 F 2 "Package_SON:Texas_PWSON-N6" H 4550 2950 50  0001 C CNN
 F 3 "" H 4550 2950 50  0001 C CNN
+F 4 "UCC27516" H 4000 3400 50  0001 C CNN "MPN"
 	1    4000 3400
 	1    0    0    -1
@@
 F 2 "Package_SON:WSON-8-1EP_2x2mm_P0.5mm_EP0.9x1.6mm_ThermalVias" H 7950 1200 50  0001 L CNN
 F 3 "http://www.ti.com/lit/ds/symlink/tps62170.pdf" H 7800 2100 50  0001 C CNN
+F 4 "TPS62172DSG" H 7800 1550 50  0001 C CNN "MPN"
 	1    7800 1550
 	1    0    0    -1
@@
 F 2 "stm32-nema17:QFN-48-1EP_7x7mm_P0.5mm_EP5.6x5.6mm_ThermalVias" H 4250 750 50  0001 R CNN
 F 3 "" H 1500 1700 50  0001 C CNN
+F 4 "STM32G431CBU" H 1950 2700 50  0001 C CNN "MPN"
 	1    1950 2700
 	1    0    0    -1
@@
 F 2 "stm32-nema17:VQFN-48_EP_6.8x6.8_Pitch0.5mm" H 8250 4500 50  0001 C CNN
 F 3 "" H 7650 2750 50  0001 C CNN
+F 4 "DRV8323RS" H 8150 4500 50  0001 C CNN "MPN"
 	1    8150 4500
 	1    0    0    -1
@@
 F 2 "Package_TO_SOT_SMD:SOT-883" H -800 2050 50  0001 C CNN
 F 3 "~" H -1000 1950 50  0001 C CNN
+F 4 "SSM3K35CTC" H -1000 1950 50  0001 C CNN "MPN"
 	1    -1000 1950
 	1    0    0    -1
@@
 F 2 "Package_TO_SOT_SMD:SOT-883" H -800 2650 50  0001 C CNN
 F 3 "~" H -1000 2550 50  0001 C CNN
+F 4 "SSM3K35CTC" H -1000 2550 50  0001 C CNN "MPN"
 	1    -1000 2550
 	1    0    0    -1
@@
 F 2 "Package_TO_SOT_SMD:SOT-883" H -800 1450 50  0001 C CNN
 F 3 "~" H -1000 1350 50  0001 C CNN
+F 4 "SSM3K35CTC" H -1000 1350 50  0001 C CNN "MPN"
 	1    -1000 1350
 	1    0    0    -1
@@
 F 2 "Resistor_SMD:R_0402_1005Metric" H 5800 5500 50  0001 C CNN
 F 3 "~" H 5800 5500 50  0001 C CNN
-F 4 "RC0402JR-07680RL" H 5800 5500 50  0001 C CNN "MPN"
+F 4 "RC0402FR-071KL" H 5800 5500 50  0001 C CNN "MPN"
 	1    5800 5500
 	-1   0    0    1
@@
 F 2 "Resistor_SMD:R_0402_1005Metric" H 5800 5150 50  0001 C CNN
 F 3 "~" H 5800 5150 50  0001 C CNN
-F 4 "RC0402JR-07680RL" H 5800 5150 50  0001 C CNN "MPN"
+F 4 "RC0402FR-071KL" H 5800 5150 50  0001 C CNN "MPN"
 	1    5800 5150
 	-1   0    0    1

Commit message: v0.3.1 board
Parts:
- M1: value Stepper_Motor_bipolar -> Motor_2_or_3_phase; footprint Connector_PinHeader_2.54mm:PinHeader_1x04_P2.54mm_Vertical -> Connector_PinHeader_2.54mm:PinHeader_1x06_P2.54mm_Vertical; symbol Motor:Stepper_Motor_bipolar -> Connector_Generic:Conn_01x06
Connections:
- net OA: now also M1.2 (Pin_2)
- net OB: now also M1.4 (Pin_4); no longer M1.2 (-)
- net OC: now also M1.5 (Pin_5), M1.6 (Pin_6); no longer M1.4
Other:
- note added: "SPI on STM32G4 would need \nan inverter on SLCK\nbecause hardware NSS \nonly works in Motorola Mode,\nbut DRV8323 needs reverse CPOL"
- note added: "USB-C in USB 2.0 compat mode"
- note added: "VDD can be 5V to 12V"
- moved on the sheet: J1, J9, R1, R2, R20, R21, R22, R3
