File: hardware/stm32-nema17-servo.kicad_sch (KiCad schematic)
At the start: 99 parts, among them J1 Conn_01x05, J2 C31-S-RA-CS1A-BK-SS, J3 TC-2050, J4 Screw_Terminal_01x02, J5 Screw_Terminal_01x02, J7 Conn_01x03, J8 Conn_01x03, J9 Conn_01x02, M1 Motor_2_or_3_phase, Q1 NVTFS5C658NL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

Commit message: tweaks to v0.4.0 hardware design
Parts:
- D1, D2: symbol Device:D_Schottky_Small_ALT -> Device:D_Schottky_Small_Filled
- D4, D5: symbol Device:D_Zener_Small_ALT -> Device:D_Zener_Small_Filled
Other:
- note added: "3V3 loads STM32G4 AS5047 DRV8323 IO UART"
Changed lines of the file:
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@@
     (effects (font (size 1.27 1.27)) (justify left bottom))
   )
+  (text "3V3 loads\nSTM32G4\nAS5047\nDRV8323 IO\nUART" (at 177.8 24.13 0)
+    (effects (font (size 1.27 1.27)) (justify left bottom))
+  )
   (text "DVDD is an output\n3.3V @ 30mA" (at 156.21 88.9 0)
     (effects (font (size 1.27 1.27)) (justify left bottom))
@@
   (symbol (lib_id "Device:C_Small") (at 29.21 29.21 0) (unit 1)
     (in_bom yes) (on_board yes)
-    (property "Reference" "C2" (id 0) (at 31.5468 28.0416 0)
+    (property "Reference" "C2" (id 0) (at 27.94 25.4 0)
       (effects (font (size 1.27 1.27)) (justify left))
     )
-    (property "Value" "100n" (id 1) (at 31.5468 30.353 0)
+    (property "Value" "100n" (id 1) (at 23.495 31.115 0)
       (effects (font (size 1.27 1.27)) (justify left))
     )
@@
   (symbol (lib_id "Device:C_Small") (at 55.88 22.86 0) (unit 1)
     (in_bom yes) (on_board yes)
-    (property "Reference" "C5" (id 0) (at 61.6966 22.86 90))
-    (property "Value" "100n" (id 1) (at 59.3852 22.86 90))
+    (property "Reference" "C5" (id 0) (at 59.055 22.86 0))
+    (property "Value" "100n" (id 1) (at 59.055 24.765 0))
     (property "Footprint" "Capacitor_SMD:C_0402_1005Metric" (id 2) (at 55.88 22.86 0)
       (effects (font (size 1.27 1.27)) hide)
@@
     (pin "2")
   )
-  (symbol (lib_id "Device:D_Schottky_Small_ALT") (at 241.3 156.21 270) (unit 1)
+  (symbol (lib_id "Device:D_Schottky_Small_Filled") (at 241.3 156.21 270) (unit 1)
     (in_bom yes) (on_board yes)
     (property "Reference" "D2" (id 0) (at 243.0272 155.0416 90)
@@
     (pin "1")
   )
-  (symbol (lib_id "Device:D_Zener_Small_ALT") (at 142.24 44.45 270) (unit 1)
+  (symbol (lib_id "Device:D_Zener_Small_Filled") (at 142.24 44.45 270) (unit 1)
     (in_bom yes) (on_board yes)
     (property "Reference" "D4" (id 0) (at 143.9672 43.2816 90)
@@
     (pin "2")
   )
-  (symbol (lib_id "Device:D_Schottky_Small_ALT") (at 41.91 153.67 180) (unit 1)
+  (symbol (lib_id "Device:D_Schottky_Small_Filled") (at 41.91 153.67 180) (unit 1)
     (in_bom yes) (on_board yes)
     (property "Reference" "D1" (id 0) (at 43.18 151.13 0)
@@
   (symbol (lib_id "Device:C_Small") (at 33.02 29.21 180) (unit 1)
     (in_bom yes) (on_board yes)
-    (property "Reference" "C3" (id 0) (at 35.3568 28.0416 0)
+    (property "Reference" "C3" (id 0) (at 31.75 25.4 0)
       (effects (font (size 1.27 1.27)) (justify right))
     )
-    (property "Value" "100n" (id 1) (at 35.3568 30.353 0)
+    (property "Value" "100n" (id 1) (at 30.48 33.02 0)
       (effects (font (size 1.27 1.27)) (justify right))
     )
@@
   (symbol (lib_id "Device:C_Small") (at 21.59 41.91 0) (unit 1)
     (in_bom yes) (on_board yes)
-    (property "Reference" "C1" (id 0) (at 23.9268 40.7416 0)
+    (property "Reference" "C1" (id 0) (at 17.145 40.64 0)
       (effects (font (size 1.27 1.27)) (justify left))
     )
-    (property "Value" "100n" (id 1) (at 23.9268 43.053 0)
+    (property "Value" "100n" (id 1) (at 14.605 43.18 0)
       (effects (font (size 1.27 1.27)) (justify left))
     )
@@
   (symbol (lib_id "Device:C_Small") (at 67.31 30.48 0) (unit 1)
     (in_bom yes) (on_board yes)
-    (property "Reference" "C6" (id 0) (at 73.1266 30.48 90))
-    (property "Value" "100n" (id 1) (at 70.8152 30.48 90))
+    (property "Reference" "C6" (id 0) (at 70.485 30.48 0))
+    (property "Value" "100n" (id 1) (at 70.485 32.385 0))
     (property "Footprint" "Capacitor_SMD:C_0402_1005Metric" (id 2) (at 67.31 30.48 0)
       (effects (font (size 1.27 1.27)) hide)
@@
       (effects (font (size 1.27 1.27)) hide)
     )
-    (property "Value" "GNDA" (id 1) (at 71.12 34.29 0))
+    (property "Value" "GNDA" (id 1) (at 69.85 36.195 0))
     (property "Footprint" "" (id 2) (at 67.31 33.02 0)
       (effects (font (size 1.27 1.27)) hide)
@@
     (pin "2")
   )
-  (symbol (lib_id "Device:D_Zener_Small_ALT") (at 165.1 44.45 270) (unit 1)
+  (symbol (lib_id "Device:D_Zener_Small_Filled") (at 165.1 44.45 270) (unit 1)
     (in_bom yes) (on_board yes)
     (property "Reference" "D5" (id 0) (at 166.8272 43.2816 90)
