File: hardware/smol-servo-tmc6200/smol-servo-tmc6200.kicad_sch (KiCad schematic)
At the start: 122 parts, among them J1 Conn_01x05, J2 C31-S-RA-CS1A-BK-SS, J3 TC-2050, J4 Screw_Terminal_01x02, J5 Screw_Terminal_01x02, J7 Conn_01x03, J8 Conn_01x03, J9 Conn_01x02, M1 Motor_2_or_3_phase, Q1 NVTFS5C658NL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

Commit message: rearrange TMC6200 version to have MCU closer to driver chip
Parts:
- added R50: 1K, Resistor_SMD:R_0402_1005Metric, symbol Device:R_Small
Connections:
- net SYNC: now also R50.1; no longer J9.2 (Pin_2)
- new net: J9.2 (Pin_2), R50.2
Changed lines of the file:
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@@
     (stroke (width 0) (type default) (color 0 0 0 0))
   )
-  (wire (pts (xy 73.66 129.54) (xy 66.04 129.54))
-    (stroke (width 0) (type default) (color 0 0 0 0))
-  )
   (wire (pts (xy -12.7 29.21) (xy -11.43 29.21))
     (stroke (width 0) (type default) (color 0 0 0 0))
@@
     (stroke (width 0) (type default) (color 0 0 0 0))
   )
+  (wire (pts (xy 73.66 127.635) (xy 73.66 129.54))
+    (stroke (width 0) (type default) (color 0 0 0 0))
+  )
   (wire (pts (xy 146.05 68.58) (xy 149.86 68.58))
     (stroke (width 0) (type default) (color 0 0 0 0))
@@
     (stroke (width 0) (type default) (color 0 0 0 0))
   )
+  (wire (pts (xy 71.12 127.635) (xy 73.66 127.635))
+    (stroke (width 0) (type default) (color 0 0 0 0))
+  )
   (wire (pts (xy 378.46 327.66) (xy 383.54 327.66))
     (stroke (width 0) (type default) (color 0 0 0 0))
@@
     )
   )
-  (global_label "SYNC" (shape input) (at 73.66 132.08 180) (fields_autoplaced)
+  (global_label "SYNC" (shape input) (at 68.58 132.08 180) (fields_autoplaced)
     (effects (font (size 1.27 1.27)) (justify right))
-    (property "Intersheet References" "${INTERSHEET_REFS}" (id 0) (at 0 0 0)
+    (property "Intersheet References" "${INTERSHEET_REFS}" (id 0) (at -5.08 0 0)
       (effects (font (size 1.27 1.27)) hide)
     )
@@
     (pin "4")
   )
-  (symbol (lib_id "power:GND") (at 66.04 129.54 0) (unit 1)
+  (symbol (lib_id "power:GND") (at 71.12 127.635 0) (unit 1)
     (in_bom yes) (on_board yes)
-    (property "Reference" "#PWR0108" (id 0) (at 66.04 135.89 0)
+    (property "Reference" "#PWR0108" (id 0) (at 71.12 133.985 0)
       (effects (font (size 1.27 1.27)) hide)
     )
-    (property "Value" "GND" (id 1) (at 63.5 132.08 0))
-    (property "Footprint" "" (id 2) (at 66.04 129.54 0)
+    (property "Value" "GND" (id 1) (at 67.31 128.905 0))
+    (property "Footprint" "" (id 2) (at 71.12 127.635 0)
       (effects (font (size 1.27 1.27)) hide)
     )
-    (property "Datasheet" "" (id 3) (at 66.04 129.54 0)
+    (property "Datasheet" "" (id 3) (at 71.12 127.635 0)
       (effects (font (size 1.27 1.27)) hide)
     )
@@
     (pin "1")
   )
+  (symbol (lib_id "Device:R_Small") (at 71.12 132.08 90) (unit 1)
+    (in_bom yes) (on_board yes)
+    (property "Reference" "R50" (id 0) (at 69.85 134.62 90)
+      (effects (font (size 1.27 1.27)) (justify left))
+    )
+    (property "Value" "1K" (id 1) (at 73.66 134.62 90)
+      (effects (font (size 1.27 1.27)) (justify left))
+    )
+    (property "Footprint" "Resistor_SMD:R_0402_1005Metric" (id 2) (at 71.12 132.08 0)
+      (effects (font (size 1.27 1.27)) hide)
+    )
+    (property "Datasheet" "~" (id 3) (at 71.12 132.08 0)
+      (effects (font (size 1.27 1.27)) hide)
+    )
+    (property "MPN" "RC0402FR-071KL" (id 4) (at 71.12 132.08 0)
+      (effects (font (size 1.27 1.27)) hide)
+    )
+    (pin "1")
+    (pin "2")
+  )
   (symbol (lib_id "power:+3.3V") (at 330.2 220.98 0) (unit 1)
     (in_bom yes) (on_board yes)
@@
       (reference "R49") (unit 1) (value "10R") (footprint "Resistor_SMD:R_0402_1005Metric")
     )
+    (path "/087ce227-67c4-4b76-be91-ef013c1af21a"
+      (reference "R50") (unit 1) (value "1K") (footprint "Resistor_SMD:R_0402_1005Metric")
+    )
     (path "/00000000-0000-0000-0000-00005d5f5911"

Commit message: v0.6.1 hardware
Parts:
- C12: MPN CC0402KRX5R8BB104 -> CL05B224KO5NNNC
- C14, C15: MPN CC0402KRX5R8BB104 -> CL05C220JB5NNNC
- C18: MPN GRM155R62A104ME14D -> CC0402KRX5R8BB104
- C20: MPN GRM155R62A104ME14D -> GRM155C80J225KE95D
- C22: footprint Capacitor_SMD:C_0402_1005Metric -> Capacitor_SMD:C_0603_1608Metric; MPN GRM155R62A104ME14D -> C1608X7R2A223K080AA
- R7: MPN RC0402FR-07100RL -> RC0402FR-07374KL
- R8: MPN RC0402FR-07100RL -> RC0402FR-07127KL
Changed lines of the file:
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@@
       (effects (font (size 1.27 1.27)) hide)
     )
-    (property "MPN" "GRM155R62A104ME14D" (id 4) (at 340.36 215.9 0)
+    (property "MPN" "GRM155C80J225KE95D" (id 4) (at 340.36 215.9 0)
       (effects (font (size 1.27 1.27)) hide)
     )
@@
       (effects (font (size 1.27 1.27)) hide)
     )
-    (property "MPN" "CC0402KRX5R8BB104" (id 4) (at 111.125 273.05 0)
+    (property "MPN" "CL05C220JB5NNNC" (id 4) (at 111.125 273.05 0)
       (effects (font (size 1.27 1.27)) hide)
     )
@@
       (effects (font (size 1.27 1.27)) hide)
     )
-    (property "MPN" "RC0402FR-07100RL" (id 4) (at 73.66 284.48 0)
+    (property "MPN" "RC0402FR-07374KL" (id 4) (at 73.66 284.48 0)
       (effects (font (size 1.27 1.27)) hide)
     )
@@
       (effects (font (size 1.27 1.27)) (justify left))
     )
-    (property "Footprint" "Capacitor_SMD:C_0402_1005Metric" (id 2) (at 356.87 198.12 0)
+    (property "Footprint" "Capacitor_SMD:C_0603_1608Metric" (id 2) (at 356.87 198.12 0)
       (effects (font (size 1.27 1.27)) hide)
     )
@@
       (effects (font (size 1.27 1.27)) hide)
     )
-    (property "MPN" "GRM155R62A104ME14D" (id 4) (at 356.87 198.12 0)
+    (property "MPN" "C1608X7R2A223K080AA" (id 4) (at 356.87 198.12 0)
       (effects (font (size 1.27 1.27)) hide)
     )
@@
       (effects (font (size 1.27 1.27)) hide)
     )
-    (property "MPN" "CC0402KRX5R8BB104" (id 4) (at 111.125 326.39 0)
+    (property "MPN" "CL05C220JB5NNNC" (id 4) (at 111.125 326.39 0)
       (effects (font (size 1.27 1.27)) hide)
     )
@@
       (effects (font (size 1.27 1.27)) hide)
     )
-    (property "MPN" "GRM155R62A104ME14D" (id 4) (at 323.85 210.82 0)
+    (property "MPN" "CC0402KRX5R8BB104" (id 4) (at 323.85 210.82 0)
       (effects (font (size 1.27 1.27)) hide)
     )
@@
       (effects (font (size 1.27 1.27)) hide)
     )
-    (property "MPN" "CC0402KRX5R8BB104" (id 4) (at 109.22 261.62 0)
+    (property "MPN" "CL05B224KO5NNNC" (id 4) (at 109.22 261.62 0)
       (effects (font (size 1.27 1.27)) hide)
     )
@@
       (effects (font (size 1.27 1.27)) hide)
     )
-    (property "MPN" "RC0402FR-07100RL" (id 4) (at 73.66 337.82 0)
+    (property "MPN" "RC0402FR-07127KL" (id 4) (at 73.66 337.82 0)
       (effects (font (size 1.27 1.27)) hide)
     )
@@
     )
     (path "/5c935e0a-78bd-4fc8-a750-5bfd4adde450"
-      (reference "C22") (unit 1) (value "22n 100V") (footprint "Capacitor_SMD:C_0402_1005Metric")
+      (reference "C22") (unit 1) (value "22n 100V") (footprint "Capacitor_SMD:C_0603_1608Metric")
     )
     (path "/00000000-0000-0000-0000-00005d56448d"

Commit message: add v0.7.0 prelim hardware design with USB Power Delivery
Parts:
- removed F1: 500mA, Fuse:Fuse_1206_3216Metric, symbol Device:Polyfuse_Small
- removed R4, R5: 5K1, Resistor_SMD:R_0402_1005Metric, symbol Device:R_Small
- added J6: Conn_01x02, Connector_PinHeader_2.54mm:PinHeader_1x02_P2.54mm_Vertical, symbol Connector_Generic:Conn_01x02
- D1: value 1A -> 5A 50V; footprint Diode_SMD:D_0402_1005Metric -> stm32-nema17:Diode-SMPA-DO-221BC; MPN CDBQT140-HF;SM5819L2-TP -> V8PAM10S-M3/H
Connections:
- net DRVEN: now also U1.4 (PC15/OSC32_OUT); no longer U1.15 (PA7)
- net DRVFAULT: now also U1.6 (PF1/OSC_OUT); no longer U1.16 (PC4)
- net ENA: now also U1.3 (PC14/OSC32_IN); no longer U1.19 (PB2)
- net ENC: now also U1.2 (PC13); no longer U1.17 (PB0)
- net ENCA: now also U1.14 (PA6); no longer U1.42 (PB4)
- net LEDB: now also U1.47 (PB9); no longer U1.44 (PB6)
- net PWMR: now also U1.15 (PA7); no longer U1.8 (PA0)
- net SOB: now also U1.19 (PB2); no longer U1.13 (PA5)
- net SOC: now also U1.16 (PC4); no longer U1.14 (PA6)
- net SYNC: now also U1.13 (PA5); no longer U1.47 (PB9)
- net VBUS: now also D1.1 (K)
- net USB_CC1: now reaches J2.A5 (CC1)
- net USB_CC1: now also U1.44 (PB6)
- net USB_CC2: now reaches J2.B5 (CC2)
- net USB_CC2: now also U1.42 (PB4)
- new net ADC1_1: J6.1 (Pin_1), U1.8 (PA0)
- new net ADC1_15: J6.2 (Pin_2), U1.17 (PB0)
- no-connect marks 18 -> 14
Other:
- note added: "USB-C in USB 2.0 compat mode but with Power Delivery"
- note removed: "USB-C in USB 2.0 compat mode"
