File: hardware/smol-servo-rp-nodrv/smol-servo-rp-nodrv.kicad_pcb (KiCad board)
At the start: 4 copper layers, 42 x 42 mm, 91 parts, among them J1 USB-C, J2 Conn_02x05_Odd_Even, J3 TC-2050, J4 Conn_02x03_Odd_Even, J5 Conn_02x05_Odd_Even, J6 Conn_02x05_Odd_Even, J7 Conn_02x05_Odd_Even, J8 Conn_01x05_Odd_Even, J9 Conn_02x05_Odd_Even, Q3 NVTFS5C658NL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

Commit message: v0.9.1 RP2350 fixes
Parts:
- removed D3, D4: 60V 500mA, Diode_SMD:D_SOD-882
- added Q4: NVTFS5C658NL, stm32-nema17:WDFN8, F.Cu at (162.5, 109.8)
- added TP1: TestPoint, TestPoint:TestPoint_Pad_D1.0mm, F.Cu at (169.0, 108.5)
- J1: value USB-C -> USB-C GT-USB-7028A
- moved Q3 1.00 mm to (162.5, 113.5)
Connections:
- C2 pad 1: VLOG -> VBUS
- U2 pad 2: VLOG -> VBUS
- U2 pad 3: VLOG -> VBUS
- U3 pad 17: unconnected-(U3-GPIO17-Pad17) -> ~{USB_PROT_FLT}
- U5 pad 17: unconnected-(U5-EPR_BLK_G-Pad17) -> EPR_BLK_G
Routing:
- net VBUS: track 35.7 -> 89.0 mm
- net VLOG: track 50.0 -> 0.00 mm
- net VUSB_LV: track 8.58 -> 38.4 mm, vias 2 -> 4
- net EPR_BLK_G: track 0.00 -> 24.5 mm, vias 0 -> 2
- net ~{USB_PROT_FLT}: track 5.92 -> 21.8 mm, vias 2 -> 5
- net VUSB: track 96.8 -> 93.4 mm, vias 17 -> 28
- net Net-(Q3-G): track 2.76 -> 1.85 mm
- net USB_CC2: track 16.7 -> 17.5 mm
- net +3V3: vias 23 -> 28
- added copper zone on B.Cu, net VUSB
Other:
- board text added: "(c) 2026-01"
- board text added: "dognotdog @gmail.com"
- board text added: "v0.9.1"
- board text removed: "(c) 2025-10"
- board text removed: "dgulyas @inrobco.de"
- board text removed: "v0.9.0"
