File: hardware/smol-servo-rp-nodrv/smol-servo-rp-nodrv.kicad_sch (KiCad schematic)
At the start: 96 parts, among them J1 USB-C, J2 Conn_02x05_Odd_Even, J3 TC-2050, J4 Conn_02x03_Odd_Even, J5 Conn_02x05_Odd_Even, J6 Conn_02x05_Odd_Even, J7 Conn_02x05_Odd_Even, J8 Conn_01x05_Odd_Even, J9 Conn_02x05_Odd_Even, Q1 BCM856BS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

Commit message: v0.9.1 RP2350 fixes
Parts:
- removed D3, D4: 60V 500mA, Diode_SMD:D_SOD-882, symbol Device:D_Schottky_Small_Filled
- added Q4: NVTFS5C658NL, stm32-nema17:WDFN8, symbol stm32-nema17:Q_NMOS_WDFN8
- added TP1: TestPoint, TestPoint:TestPoint_Pad_D1.0mm, symbol Connector:TestPoint
- C28: JLCPCB (none) -> C3909603; MPN (none) -> GMC04X7R223K100NT
- C30: JLCPCB C5137468 -> C162178; MPN CC0402KRX5R8BB104 -> GRM155R62A104KE14D
- J1: value USB-C -> USB-C GT-USB-7028A
- R32: now fitted; now in the parts list
Connections:
- net VLOG is gone; now on net VBUS: C2.1, U2.2 (EN/UVLO), U2.3 (VIN)
- net VUSB: now also Q4.5-8 (D)
- net VUSB_LV: now also Q4.1-3 (S), TP1.1
- net ~{USB_PROT_FLT}: now also U3.17 (GPIO17)
- net EPR_BLK_G: now reaches U5.17 (EPR_BLK_G)
- net EPR_BLK_G: now also Q4.4 (G)
- no-connect marks 19 -> 17
Other:
- note added: "3.3V output Fed from VBUS, which should be fed from VUSB as well."
- note added: "Looks like we need this FET for VBUS_LV to work right."
- note removed: "3.3V output Fed from both USB and VBUS to allow electronics to come up form 5V USB"
- company: InRobCo -> Dömötör Gulyas
- title: smol-servo-tmc6200 -> smol-servo-rp-ndrv
