File: hardware/smol-servo-rpi2350-tmc6200/smol-servo-rpi2350-tmc6200.kicad_pcb (KiCad board)
At the start: 4 copper layers, 48 x 44.5 mm, 148 parts, among them J11 Conn_02x10_Odd_Even, J2 C31-S-RA-CS1A-BK-SS, J3 TC-2050, J4 Screw_Terminal_01x02, J5 Screw_Terminal_01x02, M1 Motor_2_or_3_phase, Q1 NVTFS5C658NL, Q2 NVTFS5C658NL, Q3 NVTFS5C658NL, Q4 NVTFS5C658NL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

Commit message: updated RP2350 hardware
Parts:
- removed TP1, TP2: TestPoint, TestPoint:TestPoint_Pad_D1.0mm
- C2, C3: value 200p -> 220p
- U1: value RP2350_80QFN -> RP2354B
Other:
- board text added: "RESET"
- board text added: "USB BOOT"
- board text removed: "AN1 AN15"
- board text removed: "ENCODER INPUT"
- board text removed: "G V 3 I A B"
- board text removed: "GND SYNC"
- board text removed: "I2C"
- board text removed: "RX"
- board text removed: "SW1"
- board text removed: "SYNC"
- board text removed: "TX"
- board text removed: "UART"

Commit message: addition of USB-C reverse current protection
Parts:
- removed D1: 5A 50V, stm32-nema17:Diode-SMPA-DO-221BC
- added D10: 60V 500mA, Diode_SMD:D_SOD-882, F.Cu at (146.2, 130.2)
- added D11: 10V 0.3mA, Diode_SMD:D_0402_1005Metric, F.Cu at (165.8, 121.2)
- added D9: 60V 500mA, Diode_SMD:D_SOD-882, F.Cu at (144.9, 128.9)
- added Q8: DMP3013SFV, stm32-nema17:WDFN8, F.Cu at (162.6, 121.6)
- added R33: 220K, Resistor_SMD:R_0402_1005Metric, F.Cu at (167.0, 121.2)
- moved L1 8.23 mm to (161.6, 117.9), turned to 90 degrees
Connections:
- C10 pad 1: VBUS -> Net-(D10-K)
- J11 pad 11: unconnected-(J11-Pin_11-Pad11) -> GPIO8
- J11 pad 13: unconnected-(J11-Pin_13-Pad13) -> GPIO9
- U1 pad 6: unconnected-(U1-GPIO8-Pad6) -> GPIO8
- U1 pad 7: unconnected-(U1-GPIO9-Pad7) -> GPIO9
- U2 pad 2: VBUS -> Net-(D10-K)
- U2 pad 3: VBUS -> Net-(D10-K)
Routing:
- net VUSB: track 24.7 -> 45.5 mm, vias 2 -> 8
- net GPIO9: track 0.00 -> 10.9 mm, vias 0 -> 1
- net GPIO8: track 0.00 -> 10.4 mm, vias 0 -> 2
- net Net-(D10-K): track 0.00 -> 7.20 mm
- net VBUS: track 25.8 -> 22.0 mm
- net Net-(D11-A): track 0.00 -> 2.97 mm
- net GND: track 109.6 -> 111.6 mm
- net Net-(J2-SHIELD): track 23.8 -> 22.7 mm
- net USB_CC1: track 11.7 -> 12.3 mm
- added copper zone on B.Cu, net VUSB
Other:
- board text added: "240W USB PD"
- board text added: "SMOL-SERVO-RP-TMC6200 V0.8.1 (c) 2024-08 dgulyas@inrobco.de"
- board text added: "v0.8.1"
- board text removed: "SMOL-SERVO-RP-TMC6200 V0.8.0 (c) 2024-08 dgulyas@inrobco.de"
- board text removed: "v0.8.0"

Commit message: change RP2350 board to JLCPCB spec as they are the only ones who have RP2354B chips at the moment
Parts:
- removed L1: BLM18PG471SN1D, Inductor_SMD:L_0603_1608Metric
- moved C8 0.10 mm to (137.5, 110.8)
Connections:
- J2 pad S1: Net-(J2-SHIELD) -> GND
Routing:
- net Net-(J2-SHIELD): track 22.7 -> 0.00 mm
- net GND: track 111.6 -> 129.7 mm
- net VDD: track 116.8 -> 117.6 mm
- net USB_CC2: track 14.6 -> 15.1 mm
Other:
- rule pad_to_mask_clearance: 0.0254 -> 0
- rule solder_mask_min_width: 0.1016 -> 0.1

Commit message: v0.9.1 RP2350 fixes
Parts:
- added Q9: BCM856BS, Package_TO_SOT_SMD:SOT-363_SC-70-6, F.Cu at (168.8, 121.5)
- added R34: 220K, Resistor_SMD:R_0402_1005Metric, F.Cu at (166.5, 121.8)
- C12: value 220nF -> 220n
- C13: value 100nF -> 100n
- R25, R26: value 1K -> 4K7
- R54, R55: value 4.7K -> 4K7
- moved R33 1.41 mm to (166.0, 120.2), turned to 180 degrees
- moved D11 0.56 mm to (165.5, 121.8)
- moved C44 0.35 mm to (142.1, 107.2)
- moved C38 0.35 mm to (142.1, 110.2)
- moved C48 0.35 mm to (142.1, 105.2)
- turned R25 to 0 degrees
- turned R50 to 0 degrees
Connections:
- J11 pad 10: Net-(J11-Pin_10) -> SCL1_EXT
- J11 pad 12: unconnected-(J11-Pin_12-Pad12) -> GPIO12
- J11 pad 15: unconnected-(J11-Pin_15-Pad15) -> GPIO13
- J11 pad 8: Net-(J11-Pin_8) -> SDA1_EXT
- R25 pad 1: SCL3 -> SCL1_EXT
- R25 pad 2: Net-(J11-Pin_10) -> +3V3
- R26 pad 1: SDA3 -> +3V3
- R26 pad 2: Net-(J11-Pin_8) -> SDA1_EXT
- R33 pad 1: Net-(D11-A) -> Net-(Q9A-B1)
- U1 pad 11: unconnected-(U1-GPIO12-Pad11) -> GPIO12
- U1 pad 12: unconnected-(U1-GPIO13-Pad12) -> GPIO13
- U1 pad 13: unconnected-(U1-GPIO14-Pad13) -> SDA1_EXT
- U1 pad 14: unconnected-(U1-GPIO15-Pad14) -> SCL1_EXT
- U1 pad 16: unconnected-(U1-GPIO16-Pad16) -> SYNC
Routing:
- net GND: track 129.7 -> 84.0 mm, vias 104 -> 113
- net SCL1_EXT: track 0.00 -> 28.6 mm, vias 0 -> 1
- net SDA1_EXT: track 0.00 -> 25.2 mm, vias 0 -> 1
- net SYNC: track 0.00 -> 17.2 mm, vias 0 -> 2
- net Net-(J11-Pin_10): track 16.5 -> 0.00 mm, vias 1 -> 0
- net Net-(J11-Pin_8): track 13.0 -> 0.00 mm, vias 1 -> 0
- net GPIO12: track 0.00 -> 12.1 mm, vias 0 -> 3
- net GPIO13: track 0.00 -> 10.3 mm, vias 0 -> 2
- net NRST: track 29.8 -> 21.2 mm
- net VBUS: track 22.0 -> 14.1 mm, vias 101 -> 100
- net Net-(Q9A-B1): track 0.00 -> 5.81 mm
- net SWDIO: track 17.4 -> 13.8 mm
- net PWMC: track 19.4 -> 16.0 mm
- net VUSB: track 45.5 -> 48.9 mm, vias 8 -> 9
- net ENB: track 24.9 -> 21.5 mm
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Other:
- board text added: "(c) 2025-10"
- board text added: "v0.9.0"
- board text removed: "(c) 2024-08"
- board text removed: "v0.8.1"
