File: hardware/smol-servo-rpi2350-tmc6200/smol-servo-rpi2350-tmc6200.kicad_sch (KiCad schematic)
At the start: 148 parts, among them J11 Conn_02x10_Odd_Even, J2 C31-S-RA-CS1A-BK-SS, J3 TC-2050, J4 Screw_Terminal_01x02, J5 Screw_Terminal_01x02, M1 Motor_2_or_3_phase, Q1 NVTFS5C658NL, Q2 NVTFS5C658NL, Q3 NVTFS5C658NL, Q4 NVTFS5C658NL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

Commit message: updated RP2350 hardware
Parts:
- removed TP1, TP2: TestPoint, TestPoint:TestPoint_Pad_D1.0mm, symbol Connector:TestPoint
- C2, C3: value 200p -> 220p; MPN (none) -> CC0402KRX5R8BB224
- C34, C35, C36: MPN (none) -> CC0402MRX5R6BB475
- C38: MPN CC0402KRX5R8BB104 -> CC0402MRX5R6BB475
- C49, C50: MPN (none) -> CC0402JRNPO8BN150
- D6: MPN (none) -> BB-2020BGR-TRB
- H1, H2, H3, H4, J3: now left out of the parts list
- R15, R17, R19, R29, R32: MPN RC0402FR-075K11L -> RC0402FR-075K1L
- R4: MPN RC0402FR-07120KL -> RC0402FR-0733RL
- R5, R51: MPN (none) -> RC0402FR-0727RL
- R54, R55: MPN (none) -> RC0402FR-074K7L
- R56: MPN (none) -> RC0402FR-0710KL
- R57: MPN (none) -> RC0402FR-0747KL
- U1: value RP2350_80QFN -> RP2354B; MPN (none) -> RP2354B
- U2, U5: MPN (none) -> LT3990*DD
- U6: MPN (none) -> TMC6200
- U8: MPN (none) -> FUSB302BMPX
- U9: MPN (none) -> TPS71550
- Y1: MPN (none) -> ABM8-272-T3
Other:
- note removed: "Test points for otherwise unused GPIO pins"

Commit message: addition of USB-C reverse current protection
Parts:
- removed D1: 5A 50V, stm32-nema17:Diode-SMPA-DO-221BC, symbol Device:D_Schottky_Small_Filled
- added D10, D9: 60V 500mA, Diode_SMD:D_SOD-882, symbol Device:D_Schottky_Small_Filled
- added D11: 10V 0.3mA, Diode_SMD:D_0402_1005Metric, symbol Device:D_Zener_Small_Filled
- added Q8: DMP3013SFV, stm32-nema17:WDFN8, symbol Transistor_FET:DMP3013SFV
- added R33: 220K, Resistor_SMD:R_0402_1005Metric, symbol Device:R_Small
Connections:
- net GND: now also R33.2
- net VBUS: now also D10.2 (A), D11.1 (K), Q8.1-3 (S); no longer C10.1, U2.2 (EN/UVLO), U2.3 (VIN)
- net VUSB: now also D9.2 (A), Q8.5-8 (D)
- net GPIO8: now reaches J11.11 (Pin_11)
- net GPIO8: now also U1.6 (GPIO8)
- net GPIO9: now reaches J11.13 (Pin_13)
- net GPIO9: now also U1.7 (GPIO9)
- new net: D11.2 (A), Q8.4 (G), R33.1
- new net: C10.1, D10.1 (K), D9.1 (K), U2.2 (EN/UVLO), U2.3 (VIN)
- no-connect marks 25 -> 23
Other:
- note added: "3.3V output Fed from both USB and VBUS to allow electronics to come up form 5V USB"
- note added: "3V3 loads RP2354B AS5047 TMC6200 IO UART"
- note removed: "3.3V output"
- note removed: "3V3 loads STM32G4 AS5047 TMC6200 IO UART"
- moved on the sheet: C10, C12, C14, C16, J4, J5, L2, R12, R13, R7, U2

Commit message: change RP2350 board to JLCPCB spec as they are the only ones who have RP2354B chips at the moment
Parts:
- removed L1: BLM18PG471SN1D, Inductor_SMD:L_0603_1608Metric, symbol Device:L
- D11: MPN CZRQR3V3B-HF -> CZRQR10VB-HF;PZU10B2L,315
- D2: MPN CZRU52C20 -> CZRU52C20;BZX584B20V
- L5: MPN (none) -> AOTA-B201610S3R3-101-T
Connections:
- net GND: now also J2.S1 (SHIELD)
Changed lines of the file:
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@@
 (kicad_sch
-	(version 20231120)
+	(version 20250114)
 	(generator "eeschema")
-	(generator_version "8.0")
+	(generator_version "9.0")
 	(paper "A2")
 	(title_block
@@
 		(company "InRobCo")
 	)
+	(text "3.3V output\nFed from both USB and VBUS to allow electronics to come up form 5V USB"
+		(exclude_from_sim no)
+		(at 162.56 260.985 0)
+		(effects
+			(font
+				(size 1.27 1.27)
+			)
+			(justify left bottom)
+		)
+	)
+	(text "Additional caps on VBUS"
+		(exclude_from_sim no)
+		(at 216.535 74.295 0)
+		(effects
+			(font
+				(size 1.27 1.27)
+			)
+			(justify left bottom)
+		)
+	)
+	(text "maybe STUSB1602/PTN5110 would work for USB PD\nFUSB302BMPX seems smallest"
+		(exclude_from_sim no)
+		(at 464.185 22.86 0)
+		(effects
+			(font
+				(size 1.27 1.27)
+			)
+			(justify left bottom)
+		)
+	)
+	(text "4937N (30V) can do 8A continuous current on minimal pad in thermal limit\nNVTFS5C658NL is a similar 60V part"
+		(exclude_from_sim no)
+		(at 250.825 288.925 0)
+		(effects
+			(font
+				(size 1.27 1.27)
+			)
+			(justify left bottom)
+		)
+	)
+	(text "12V output"
+		(exclude_from_sim no)
+		(at 160.655 318.77 0)
+		(effects
+			(font
+				(size 1.27 1.27)
+			)
+			(justify left bottom)
+		)
+	)
+	(text "3V3 loads\nRP2354B\nAS5047\nTMC6200 IO\nUART"
+		(exclude_from_sim no)
+		(at 206.375 273.05 0)
+		(effects
+			(font
+				(size 1.27 1.27)
+			)
+			(justify left bottom)
+		)
+	)
+	(text "Analog\n3x Current Sense (SOx)\nVBUS\nVDD\n3x Aux / Bridge Voltage"
+		(exclude_from_sim no)
+		(at 446.405 190.5 0)
+		(effects
+			(font
+				(size 1.27 1.27)
+			)
+			(justify left bottom)
+		)
+	)
+	(text "SPI0:\n  AD5047\nSPI1:\n  TMC6200\nUART1: \n  DBG / console\nI2C0:\n  FUSB302\nPWM8:\n  PWMC\n  ENC\nPIO0:\n  LED_CLK\n  LED_MOSI\nPIO1:\n  ENCA\n  ENCB\n  ENCI\nPIO2:\n  PWMx/ENx"
+		(exclude_from_sim no)
+		(at 458.47 92.71 0)
+		(effects
+			(font
+				(size 1.27 1.27)
+			)
+			(justify left bottom)
+		)
+	)
+	(text "Gate Resistors might need higher values for low C_g MOSFETS\nto avoid to fast switching and induced ringing."
+		(exclude_from_sim no)
+		(at 485.775 373.38 0)
+		(effects
+			(font
+				(size 1.27 1.27)
+			)
+			(justify left bottom)
+		)
+	)
+	(text "V0.2: VBUS feedback"
+		(exclude_from_sim no)
+		(at 213.995 46.355 0)
+		(effects
+			(font
+				(size 1.27 1.27)
+			)
+			(justify left bottom)
+		)
+	)
+	(text "SPI on STM32G4 would need \nan inverter on SLCK\nbecause hardware NSS \nonly works in Motorola Mode,\nbut DRV8323 needs reverse CPOL"
+		(exclude_from_sim no)
+		(at 213.995 120.015 0)
+		(effects
+			(font
+				(size 1.27 1.27)
+			)
+			(justify left bottom)
+		)
+	)
+	(text "clamp VBUS sense to 20V, \n48V ops is not supported"
+		(exclude_from_sim no)
+		(at 542.29 76.454 0)
+		(effects
+			(font
+				(size 1.27 1.27)
+			)
+			(justify left bottom)
+		)
+	)
+	(text "on Circuithub stackup (R=4.7,h=0.2mm)\nuse 12mil wide w/ 4mil spacing for D+/D- pair"
+		(exclude_from_sim no)
+		(at 68.58 188.595 0)
+		(effects
+			(font
+				(size 1.27 1.27)
+			)
+			(justify left bottom)
+		)
+	)
+	(text "LED has a 5V LDO supply"
+		(exclude_from_sim no)
+		(at 52.705 38.735 0)
+		(effects
+			(font
+				(size 1.27 1.27)
+			)
+			(justify left bottom)
+		)
+	)
+	(text "additional bridge voltage sensing for sensorless FOC"
+		(exclude_from_sim no)
+		(at 490.22 153.035 0)
+		(effects
+			(font
+				(size 1.27 1.27)
+			)
+			(justify left bottom)
+		)
+	)
+	(text "USB-C in USB 2.0 compat mode\nbut with Power Delivery"
+		(exclude_from_sim no)
+		(at 25.4 262.89 0)
+		(effects
+			(font
+				(size 1.27 1.27)
+			)
+			(justify left bottom)
+		)
+	)
 	(junction
 		(at 417.83 35.56)
@@
 	)
 	(junction
+		(at 38.1 207.01)
+		(diameter 0)
+		(color 0 0 0 0)
+	)
+	(junction
 		(at 453.39 40.64)
 		(diameter 0)
@@
 	)
 	(junction
-		(at 38.1 207.01)
-		(diameter 0)
-		(color 0 0 0 0)
-	)
-	(junction
 		(at 154.305 323.215)
 		(diameter 0)
@@
 	(wire
 		(pts
+			(xy 30.48 207.01) (xy 38.1 207.01)
+		)
+		(stroke
+			(width 0)
+			(type default)
+		)
+	)
+	(wire
+		(pts
 			(xy 516.89 325.12) (xy 518.16 325.12)
 		)
@@
 		)
 	)
-	(text "3.3V output\nFed from both USB and VBUS to allow electronics to come up form 5V USB"
-		(exclude_from_sim no)
-		(at 162.56 260.985 0)
-		(effects
-			(font
-				(size 1.27 1.27)
-			)
-			(justify left bottom)
-		)
-	)
-	(text "Additional caps on VBUS"
-		(exclude_from_sim no)
-		(at 216.535 74.295 0)
-		(effects
-			(font
-				(size 1.27 1.27)
-			)
-			(justify left bottom)
-		)
-	)
-	(text "maybe STUSB1602/PTN5110 would work for USB PD\nFUSB302BMPX seems smallest"
-		(exclude_from_sim no)
-		(at 464.185 22.86 0)
-		(effects
-			(font
-				(size 1.27 1.27)
-			)
-			(justify left bottom)
-		)
-	)
-	(text "4937N (30V) can do 8A continuous current on minimal pad in thermal limit\nNVTFS5C658NL is a similar 60V part"
-		(exclude_from_sim no)
-		(at 250.825 288.925 0)
-		(effects
-			(font
-				(size 1.27 1.27)
-			)
-			(justify left bottom)
-		)
-	)
-	(text "12V output"
-		(exclude_from_sim no)
-		(at 160.655 318.77 0)
-		(effects
-			(font
-				(size 1.27 1.27)
-			)
-			(justify left bottom)
-		)
-	)
-	(text "3V3 loads\nRP2354B\nAS5047\nTMC6200 IO\nUART"
-		(exclude_from_sim no)
-		(at 206.375 273.05 0)
-		(effects
-			(font
-				(size 1.27 1.27)
-			)
-			(justify left bottom)
-		)
-	)
-	(text "Analog\n3x Current Sense (SOx)\nVBUS\nVDD\n3x Aux / Bridge Voltage"
-		(exclude_from_sim no)
-		(at 446.405 190.5 0)
-		(effects
-			(font
-				(size 1.27 1.27)
-			)
-			(justify left bottom)
-		)
-	)
-	(text "SPI0:\n  AD5047\nSPI1:\n  TMC6200\nUART1: \n  DBG / console\nI2C0:\n  FUSB302\nPWM8:\n  PWMC\n  ENC\nPIO0:\n  LED_CLK\n  LED_MOSI\nPIO1:\n  ENCA\n  ENCB\n  ENCI\nPIO2:\n  PWMx/ENx"
-		(exclude_from_sim no)
-		(at 458.47 92.71 0)
-		(effects
-			(font
-				(size 1.27 1.27)
-			)
-			(justify left bottom)
-		)
-	)
-	(text "Gate Resistors might need higher values for low C_g MOSFETS\nto avoid to fast switching and induced ringing."
-		(exclude_from_sim no)
-		(at 485.775 373.38 0)
-		(effects
-			(font
-				(size 1.27 1.27)
-			)
-			(justify left bottom)
-		)
-	)
-	(text "V0.2: VBUS feedback"
-		(exclude_from_sim no)
-		(at 213.995 46.355 0)
-		(effects
-			(font
-				(size 1.27 1.27)
-			)
-			(justify left bottom)
-		)
-	)
-	(text "SPI on STM32G4 would need \nan inverter on SLCK\nbecause hardware NSS \nonly works in Motorola Mode,\nbut DRV8323 needs reverse CPOL"
-		(exclude_from_sim no)
-		(at 213.995 120.015 0)
-		(effects
-			(font
-				(size 1.27 1.27)
-			)
-			(justify left bottom)
-		)
-	)
-	(text "clamp VBUS sense to 20V, 48V ops is not supported"
-		(exclude_from_sim no)
-		(at 502.92 69.215 0)
-		(effects
-			(font
-				(size 1.27 1.27)
-			)
-			(justify left bottom)
-		)
-	)
-	(text "on Circuithub stackup (R=4.7,h=0.2mm)\nuse 12mil wide w/ 4mil spacing for D+/D- pair"
-		(exclude_from_sim no)
-		(at 68.58 188.595 0)
-		(effects
-			(font
-				(size 1.27 1.27)
-			)
-			(justify left bottom)
-		)
-	)
-	(text "LED has a 5V LDO supply"
-		(exclude_from_sim no)
-		(at 52.705 38.735 0)
-		(effects
-			(font
-				(size 1.27 1.27)
-			)
-			(justify left bottom)
-		)
-	)
-	(text "additional bridge voltage sensing for sensorless FOC"
-		(exclude_from_sim no)
-		(at 490.22 153.035 0)
-		(effects
-			(font
-				(size 1.27 1.27)
-			)
-			(justify left bottom)
-		)
-	)
-	(text "USB-C in USB 2.0 compat mode\nbut with Power Delivery"
-		(exclude_from_sim no)
-		(at 25.4 262.89 0)
-		(effects
-			(font
-				(size 1.27 1.27)
-			)
-			(justify left bottom)
-		)
-	)
 	(label "~{USB_BOOT}"
 		(at 326.39 83.82 0)
-		(fields_autoplaced yes)
 		(effects
 			(font
@@
 	)
 	(symbol
-		(lib_id "Device:L")
-		(at 34.29 207.01 90)
-		(unit 1)
-		(exclude_from_sim no)
-		(in_bom yes)
-		(on_board yes)
-		(dnp no)
-		(property "Reference" "L1"
-			(at 34.29 208.28 90)
-			(effects
-				(font
-					(size 1.27 1.27)
-				)
-			)
-		)
-		(property "Value" "BLM18PG471SN1D"
-			(at 49.53 207.01 90)
-			(effects
-				(font
-					(size 1.27 1.27)
-				)
-			)
-		)
-		(property "Footprint" "Inductor_SMD:L_0603_1608Metric"
-			(at 34.29 207.01 0)
-			(effects
-				(font
-					(size 1.27 1.27)
-				)
-				(hide yes)
-			)
-		)
-		(property "Datasheet" "~"
-			(at 34.29 207.01 0)
-			(effects
-				(font
-					(size 1.27 1.27)
-				)
-				(hide yes)
-			)
-		)
-		(property "Description" ""
-			(at 34.29 207.01 0)
-			(effects
-				(font
-					(size 1.27 1.27)
-				)
-				(hide yes)
-			)
-		)
-		(property "MPN" "BLM18PG471SN1D"
-			(at 34.29 207.01 0)
-			(effects
-				(font
-					(size 1.27 1.27)
-				)
-				(hide yes)
-			)
-		)
-		(pin "1"
-		)
-		(pin "2"
-		)
-		(instances
-			(project ""
-				(path "/f9c81c26-f253-4227-a69f-53e64841cfbe"
-					(reference "L1")
-					(unit 1)
-				)
-			)
-		)
-	)
-	(symbol
 		(lib_id "Connector_Generic:Conn_01x06")
 		(at 326.39 316.23 0)
@@
 			)
 		)
-		(property "MPN" "CZRQR3V3B-HF"
+		(property "MPN" "CZRQR10VB-HF;PZU10B2L,315"
 			(at 97.79 167.64 0)
 			(effects
@@
 			)
 		)
-		(property "MPN" "CZRU52C20"
+		(property "MPN" "CZRU52C20;BZX584B20V"
 			(at 554.99 88.9 90)
 			(effects
@@
 			)
 		)
-		(property "MPN" ""
+		(property "MPN" "AOTA-B201610S3R3-101-T"
 			(at 342.9 71.12 0)
 			(effects
@@
 		)
 	)
+	(embedded_fonts no)
 )

Commit message: v0.9.1 RP2350 fixes
Parts:
- added Q9: BCM856BS, Package_TO_SOT_SMD:SOT-363_SC-70-6, symbol Transistor_BJT:BC856BS
- added R34: 220K, Resistor_SMD:R_0402_1005Metric, symbol Device:R_Small
- C1, C18, C19, C21, C37, C39, C40, C41, C42, C43, C44, C45, C46, C47, C48, C8, C9: JLCPCB (none) -> C5137468
- C10, C11: JLCPCB (none) -> C2981733
- C12: value 220nF -> 220n; JLCPCB (none) -> C16772
- C13: value 100nF -> 100n; JLCPCB (none) -> C5137468
- C14, C15: JLCPCB (none) -> C1555
- C16, C17: JLCPCB (none) -> C84419
- C2, C3: JLCPCB (none) -> C39122
- C20: JLCPCB (none) -> C12530
- C22: JLCPCB (none) -> C376821
- C23, C24, C25, C31, C32, C33, C7: JLCPCB (none) -> C5156756
- C26: JLCPCB (none) -> C162178
- C27: JLCPCB (none) -> C36911431
- C28, C29, C30: JLCPCB (none) -> C29266
- C34, C35, C36, C38: JLCPCB (none) -> C23733
- C4: JLCPCB (none) -> C14445
- C49, C50: JLCPCB (none) -> C106997
- D10, D9: JLCPCB (none) -> C552935
- D11: JLCPCB (none) -> C553572
- D2: JLCPCB (none) -> C968162
- D3, D4, D5, D7, D8: JLCPCB (none) -> C3013401
- D6: JLCPCB (none) -> C22439302
- J2: JLCPCB (none) -> C6582279
- L2, L4: JLCPCB (none) -> C2849475
- L5: JLCPCB (none) -> C42411119
- Q1, Q2, Q3, Q4, Q5, Q6, Q7: JLCPCB (none) -> C5208924
- Q8: value DMP3013SFV -> 48V PFET
- R1, R2, R3: JLCPCB (none) -> C25130
- R10, R11, R9: JLCPCB (none) -> C875584
- R12, R30: JLCPCB (none) -> C26083
- R13: JLCPCB (none) -> C27012
- R14, R16, R18, R28: JLCPCB (none) -> C25750
- R15, R17, R19, R29, R32: JLCPCB (none) -> C25905
- R20, R21, R22, R23, R24, R50: JLCPCB (none) -> C11702
- R25, R26: value 1K -> 4K7; JLCPCB (none) -> C25900; MPN RC0402FR-071KL -> RC0402FR-074K7L
- R27: JLCPCB (none) -> C25741
- R31: JLCPCB (none) -> C25768
- R33: JLCPCB (none) -> C25767
- R35: JLCPCB (none) -> C25746
- R36, R57: JLCPCB (none) -> C25792
- R37, R38, R39, R40, R42, R43, R44, R46, R47, R48: JLCPCB (none) -> C17168
- R4: JLCPCB (none) -> C25105
- R41, R45, R49: JLCPCB (none) -> C102766
- R5, R51: JLCPCB (none) -> C25100
- R52, R53: JLCPCB (none) -> C11702; MPN RC0402FR-07120KL -> RC0402FR-071KL
- R54, R55: value 4.7K -> 4K7; JLCPCB (none) -> C25900
- R56: JLCPCB (none) -> C25744
- R6: JLCPCB (none) -> C25101
- R7: JLCPCB (none) -> C25781
- R8: JLCPCB (none) -> C11688
- SW1, SW2: JLCPCB (none) -> C4365176
- U1: JLCPCB (none) -> C39843328
- U2, U5: JLCPCB (none) -> C580169
- U3: JLCPCB (none) -> C3655221
- U4: now not fitted
- U6: JLCPCB (none) -> C465958
- U8: JLCPCB (none) -> C132291
- U9: JLCPCB (none) -> C571193
- Y1: JLCPCB (none) -> C20625731
Connections:
- net SCL3 is gone; now on net SCL1_EXT: R25.1
- net SDA3 is gone; now on net +3V3: R26.1
- net +3V3: now also R25.2
- net GND: now also R34.2
- net SYNC: now also U1.16 (GPIO16)
- net VBUS: now also Q9.6 (C1)
- net VUSB: now also Q9.3 (C2)
- net SCL1_EXT: now reaches J11.10 (Pin_10)
- net SCL1_EXT: now also U1.14 (GPIO15); no longer R25.2
- net SDA1_EXT: now reaches J11.8 (Pin_8), R26.2
- net SDA1_EXT: now also U1.13 (GPIO14)
- net GPIO12: now reaches J11.12 (Pin_12)
- net GPIO12: now also U1.11 (GPIO12)
- net GPIO13: now reaches J11.15 (Pin_15)
- net GPIO13: now also U1.12 (GPIO13)
- net at D11.2 (A), Q8.4 (G): now also Q9.1 (E1), R34.1; no longer R33.1
- new net: Q9.2 (B1), Q9.4 (E2), Q9.5 (B2), R33.1
- no-connect marks 23 -> 27
Other:
- note added: "P-FET switch with reverse polarity protection via bipolar comparator"
- moved on the sheet: C10, C11, C12, C13, C14, C15, C16, C17, C23, C24, C25, C31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
